Commit message: Overwrite with latest local erp42_ws

File: src/erp42_description/urdf/erp42.urdf.xacro (robot description, xacro)
@@ -1,8 +1,8 @@
 <?xml version="1.0"?>
 <robot name="erp42" xmlns:xacro="http://ros.org/wiki/xacro">
-  <xacro:arg name="pkg_share"        default=""/>
+  <xacro:arg name="pkg_share" default=""/>
   <xacro:arg name="controllers_file" default=""/>
   <xacro:include filename="$(arg pkg_share)/urdf/macros_erp42.xacro"/>
-  <!--XXXXXXXXXXXXXXXXXXXXXXXXXXXXXXXXXXXX-OK-XXXXXXXXXXXXXXXXXXXXXXXXXXXXXXXXXXXXXXXXXXXXXXXX -->
+  <xacro:include filename="$(arg pkg_share)/urdf/erp42_control.gazebo" />
   <link name="structure">
     <visual name="visual">
@@ -14,8 +14,7 @@
     <collision>
       <geometry>
-      <!--<box size=" 1.0 1.0 0.2"/>-->
-      <mesh filename="$(arg pkg_share)/meshes/erp42_structure.dae" scale="1 1 1"/>
-      </geometry>
-         <origin xyz="0 0 -0.03" rpy=" 0 0 3.14" />
+        <mesh filename="$(arg pkg_share)/meshes/erp42_structure.dae" scale="1 1 1"/>
+      </geometry>
+      <origin xyz="0 0 -0.03" rpy="0 0 3.14" />
     </collision>
     <inertial>
@@ -25,63 +24,78 @@
     </inertial>
   </link>
-<!--XXXXXXXXXXXXXXXXXXXXXXXXXXXXXXXXXXXXXXXXXXXXXXXXXXXXXXXXXXXXXXXXXXXXXXXXXXXXXXXXXXXX -->
-<!-- XXXXXXXXXXXXXXXXXXXXXXXXXXXXXXXXXXXXxXXXXXX  LINK  XXXXXXXXXxXXXXXXXXXXXXXXXXXXXXXXXXXXXXXXXXXXXXXXXX-->
+  <!-- steering links with visual for debug -->
+  <link name="lf_front_steer_link">
+    <inertial>
+      <mass value="0.1"/>
+      <origin xyz="0 0 0" rpy="0 0 0"/>
+      <inertia ixx="0.001" ixy="0" ixz="0" iyy="0.001" iyz="0" izz="0.001"/>
+    </inertial>
+    <visual>
+      <origin xyz="0 0 0" rpy="0 0 0"/>
+      <geometry>
+        <box size="0.05 0.05 0.02"/>
+      </geometry>
+      <material name="steer_green">
+        <color rgba="0 1 0 0.5"/>
+      </material>
+    </visual>
+  </link>
+  <link name="rf_front_steer_link">
+    <inertial>
+      <mass value="0.1"/>
+      <origin xyz="0 0 0" rpy="0 0 0"/>
+      <inertia ixx="0.001" ixy="0" ixz="0" iyy="0.001" iyz="0" izz="0.001"/>
+    </inertial>
+    <visual>
+      <origin xyz="0 0 0" rpy="0 0 0"/>
+      <geometry>
+        <box size="0.05 0.05 0.02"/>
+      </geometry>
+      <material name="steer_blue">
+        <color rgba="0 0 1 0.5"/>
+      </material>
+    </visual>
+  </link>
+  <!-- steering hinge joints -->
+  <joint name="lf_steering_hinge_joint" type="revolute">
+    <parent link="structure"/>
+    <child link="lf_front_steer_link"/>
+    <origin xyz="0.53 0.51 0" rpy="0 0 0"/>
+    <axis xyz="0 0 1"/>
+    <limit lower="-0.52" upper="0.52" effort="5.0" velocity="1.0"/>
+    <dynamics damping="0.1" friction="0.1"/>
+  </joint>
+  <joint name="rf_steering_hinge_joint" type="revolute">
+    <parent link="structure"/>
+    <child link="rf_front_steer_link"/>
+    <origin xyz="0.53 -0.51 0" rpy="0 0 0"/>
+    <axis xyz="0 0 1"/>
+    <limit lower="-0.52" upper="0.52" effort="5.0" velocity="1.0"/>
+    <dynamics damping="0.1" friction="0.1"/>
+  </joint>
+  <!-- front wheels (under steer links) -->
   <xacro:wheel prefix="right" suffix="front" x="0" y="0" z="0" pitch="0" yaw="1.5707"/>
+  <xacro:wheel prefix="left" suffix="front" x="0" y="0" z="0" pitch="0" yaw="-1.5707"/>
+  <xacro:wheel_joint prefix="right" suffix="front" parent_link="rf_front_steer_link" x="0" y="0" z="0"/>
+  <xacro:wheel_joint prefix="left" suffix="front" parent_link="lf_front_steer_link" x="0" y="0" z="0"/>
+  <!-- rear disk wheels and driven wheels -->
+  <xacro:disk_wheel prefix="right" suffix="back" roll="0" pitch="0" yaw="1.5707"/>
+  <xacro:disk_wheel prefix="left" suffix="back" roll="0" pitch="0" yaw="-1.5707" with_gazebo="true"/>
+  <xacro:back_disk_wheel_joint prefix="right" suffix="back" x="-0.49" y="0.51" z="0"/>
+  <xacro:back_disk_wheel_joint prefix="left" suffix="back" x="-0.49" y="-0.51" z="0"/>
   <xacro:wheel prefix="right" suffix="back" x="0" y="0" z="0" pitch="0" yaw="1.5707"/>
-  <xacro:wheel prefix="left" suffix="front" x="0" y="0" z="0" pitch="3.1414" yaw="1.5707"/>
-  <xacro:wheel prefix="left" suffix="back" x="0" y="0" z="0" pitch="3.1414" yaw="1.5707"/>
-  <!-- XXXXXXXXXXXXXXXXXXXXXXXXXXXXXXXXXXXXXXXX  DISK LINK  XXXXXXXXXXXXXXXXXXXXXXXXXXXXXXXXXXXXXXXXXXXXXX-->
-  <xacro:disk_wheel prefix="right" suffix="front" roll="0" pitch="0" yaw="1.5707"/>  <!--yall value is only for visual -->
-  <xacro:disk_wheel prefix="left" suffix="front" roll="0" pitch="0" yaw="-1.5707"/>  <!--yall value is only for visual -->
-  <xacro:disk_wheel prefix="right" suffix="back" roll="0" pitch="0" yaw="1.5707"/>  <!--yall value is only for visual -->
-  <xacro:disk_wheel prefix="left" suffix="back" roll="0" pitch="0" yaw="-1.5707" with_gazebo="true"/>  <!--yall value is only for visual -->
-  <!-- XXXXXXXXXXXXXXXXXXXXXXXXXXXXXXXXXXXXXXX  actuator  1  2   XXXXXXXXXXXXXXXXXXXXXXXXXXXXXXXXXXXXXXXXX-->
-  <xacro:wheel_joint prefix="right" suffix="front" x="0" y="0.08" z="0" /> <!--rotation in y axes, wheel connect with the front disk-->
-  <xacro:wheel_joint prefix="left" suffix="front" x="0" y="-0.08" z="0"/>  <!--rotation in y axes, wheel connect with the front disk-->
-  <!-- XXXXXXXXXXXXXXXXXXXXXXXXXXXXXXXXXXXXXXX  actuator  3  4   XXXXXXXXXXXXXXXXXXXXXXXXXXXXXXXXXXXXXXXX-->
-  <xacro:wheel_joint prefix="right" suffix="back" x="0" y="0.08" z="0" />   <!--rotation in y axes wheel connect with the back disk-->
-  <xacro:wheel_joint prefix="left" suffix="back" x="0" y="-0.08" z="0" />   <!--rotation in y axes wheel connect with the back disk-->
-  <!-- XXXXXXXXXXXXXXXXXXXXXXXXXXXXXXXXXXXXXXXXX  actuator 5 6  XXXXXXXXXXXXXXXXXXXXXXXXXXXXXXXXXXXXXXXXXX-->
-  <xacro:front_disk_wheel_joint prefix="right" suffix="front" x="0.53" y="0.51" z="0"/>  <!--disk rotation in z axes, disk connect with structure-->
-  <xacro:front_disk_wheel_joint prefix="left"  suffix="front" x="0.53" y="-0.51" z="0"/> <!--disk rotation in z axes, disk connect with structure-->
-  <!-- XXXXXXXXXXXXXXXXXXXXXXXXXXXXXXXXXXXXXXXXX  fixed  XXXXXXXXXXXXXXXXXXXXXXXXXXXXXXXXXXXXXXXXXX-->
-  <xacro:back_disk_wheel_joint prefix="right" suffix="back" x="-0.49" y="0.51" z="0"/>  <!--disk rotation in z axes, disk connect with structure-->
-  <xacro:back_disk_wheel_joint prefix="left" suffix="back" x="-0.49" y="-0.51" z="0"/> <!--disk rotation in z axes, disk connect with structure-->
-  <xacro:my_camera prefix="middle" /> <!-- camera link we cant use the name camera due to create a confuse with gazebo and presente the problem with
-	invalided parameter name-->
-  <xacro:my_camera prefix="right" /> <!-- camera link we cant use the name camera due to create a confuse with gazebo and presente the problem with
-	invalided parameter name-->
-  <xacro:my_camera prefix="left" /> <!-- camera link we cant use the name camera due to create a confuse with gazebo and presente the problem with
-	invalided parameter name-->
-  <xacro:my_camera prefix="back" /> <!-- camera link we cant use the name camera due to create a confuse with gazebo and presente the problem with
-	invalided parameter name-->
-  <xacro:camera_joint prefix="middle" x="1.0" y="0" z="0.3" roll="0" pitch="0" yaw="0"/> <!--camera joint-->
-  <xacro:camera_joint prefix="left" x="0.05" y="0.10" z="0.3" roll="0" pitch="0" yaw="0.785"/> <!--camera joint-->
-  <xacro:camera_joint prefix="right" x="0.05" y="-0.10" z="0.3" roll="0" pitch="0" yaw="-0.785"/> <!--camera joint-->
-  <xacro:camera_joint prefix="back" x="-0.05" y="0" z="0.4" roll="0" pitch="0" yaw="3.1414"/> <!--camera joint-->
-  <gazebo>
-    <plugin name="skid_steer_drive_controller" filename="libgazebo_ros_diff_drive.so">
-      <ros>
-        <namespace>/</namespace>
-        <argument>/cmd_vel:=cmd_vel</argument>
-        <argument>/odom:=odom</argument>
-      </ros>
-      <update_rate>100.0</update_rate>
-      <num_wheel_pairs>2</num_wheel_pairs>
-      <odometry_frame>odom</odometry_frame>
-      <left_joint>left_front_wheel_joint</left_joint>
-      <left_joint>left_back_wheel_joint</left_joint>
-      <right_joint>right_front_wheel_joint</right_joint>
-      <right_joint>right_back_wheel_joint</right_joint>
-      <wheel_separation>1.02</wheel_separation>
-      <wheel_diameter>0.56</wheel_diameter>
-      <robot_base_frame>structure</robot_base_frame>
-      <max_wheel_torque>15</max_wheel_torque>
-      <publish_odom>true</publish_odom>
-      <publish_odom_tf>true</publish_odom_tf>
-      <publish_wheel_tf>false</publish_wheel_tf>
-    </plugin>
-  </gazebo>
-<!-- left_camera -->
+  <xacro:wheel prefix="left" suffix="back" x="0" y="0" z="0" pitch="0" yaw="-1.5707"/>
+  <xacro:wheel_joint prefix="right" suffix="back" parent_link="right_back_disk_wheel" x="0" y="0" z="0"/>
+  <xacro:wheel_joint prefix="left" suffix="back" parent_link="left_back_disk_wheel" x="0" y="0" z="0"/>
+  <!-- cameras -->
+  <xacro:my_camera prefix="middle"/>
+  <xacro:my_camera prefix="right"/>
+  <xacro:my_camera prefix="left"/>
+  <xacro:my_camera prefix="back"/>
+  <xacro:camera_joint prefix="middle" x="1.0" y="0" z="0.3" roll="0" pitch="0" yaw="0"/>
+  <xacro:camera_joint prefix="left" x="0.05" y="0.10" z="0.3" roll="0" pitch="0" yaw="0.785"/>
+  <xacro:camera_joint prefix="right" x="0.05" y="-0.10" z="0.3" roll="0" pitch="0" yaw="-0.785"/>
+  <xacro:camera_joint prefix="back" x="-0.05" y="0" z="0.4" roll="0" pitch="0" yaw="3.1414"/>
+  <!-- camera plugins -->
   <gazebo reference="left_camera">
     <sensor type="camera" name="left_camera1">
@@ -95,7 +109,4 @@
           <noise>
             <type>gaussian</type>
-          <!-- Noise is sampled independently per pixel on each frame.
-               That pixel's noise value is added to each of its color
-               channels, which at that point lie in the range [0,1]. -->
             <mean>0.0</mean>
             <stddev>0.007</stddev>
@@ -123,5 +134,4 @@
     </sensor>
   </gazebo>
-<!-- right_camera -->
   <gazebo reference="right_camera">
     <sensor type="camera" name="right_camera2">
@@ -135,7 +145,4 @@
           <noise>
             <type>gaussian</type>
-          <!-- Noise is sampled independently per pixel on each frame.
-               That pixel's noise value is added to each of its color
-               channels, which at that point lie in the range [0,1]. -->
             <mean>0.0</mean>
             <stddev>0.007</stddev>
@@ -163,20 +170,15 @@
     </sensor>
   </gazebo>
-<!-- middle_camera -->
   <gazebo reference="middle_camera">
     <sensor type="camera" name="middle_camera3">
-      <pose>0 0 0 0 0 0</pose>
-      <update_rate>30.0</update_rate>
-      <camera name="head">
-        <horizontal_fov>1.3962634</horizontal_fov>
-        <image>
-          <width>800</width>
-          <height>800</height>
-          <format>R8G8B8</format>
-          <noise>
-            <type>gaussian</type>
-          <!-- Noise is sampled independently per pixel on each frame.
-               That pixel's noise value is added to each of its color
-               channels, which at that point lie in the range [0,1]. -->
+      <update_rate>30.0</update_rate>
+      <camera name="head">
+        <horizontal_fov>1.3962634</horizontal_fov>
+        <image>
+          <width>800</width>
+          <height>800</height>
+          <format>R8G8B8</format>
+          <noise>
+            <type>gaussian</type>
             <mean>0.0</mean>
             <stddev>0.007</stddev>
@@ -204,5 +206,4 @@
     </sensor>
   </gazebo>
-<!-- back_camera -->
   <gazebo reference="back_camera">
     <sensor type="camera" name="back_camera4">
@@ -216,7 +217,4 @@
           <noise>
             <type>gaussian</type>
-            <!-- Noise is sampled independently per pixel on each frame.
-               That pixel's noise value is added to each of its color
-               channels, which at that point lie in the range [0,1]. -->
             <mean>0.0</mean>
             <stddev>0.007</stddev>

File: src/erp42_description/urdf/macros_erp42.xacro (robot description, xacro)
@@ -12,4 +12,16 @@
   <xacro:property name="camera_size" value="0.05"/>
   <xacro:property name="camera_mass" value="1e-5"/>
+  <!-- Steering link + hinge joint for front wheels -->
+  <xacro:macro name="steer_link" params="side y_offset">
+    <link name="${side}_front_steer_link"/>
+    <joint name="${side}_steering_hinge_joint" type="revolute">
+      <parent link="structure"/>
+      <child link="${side}_front_steer_link"/>
+      <origin xyz="0 ${y_offset} 0" rpy="0 0 0"/>
+      <axis xyz="0 0 1"/>
+      <limit lower="-0.52" upper="0.52" effort="5.0" velocity="1.0"/>
+      <dynamics damping="0.1" friction="0.1"/>
+    </joint>
+  </xacro:macro>
   <!-- Wheel link -->
   <xacro:macro name="wheel" params="prefix suffix x y z pitch yaw">
@@ -34,9 +46,9 @@
     </link>
   </xacro:macro>
-  <!-- Wheel joint -->
-  <xacro:macro name="wheel_joint" params="prefix suffix x y z">
+  <!-- Wheel joint: parent_link을 인자로 받도록 변경 -->
+  <xacro:macro name="wheel_joint" params="prefix suffix parent_link x y z">
     <joint name="${prefix}_${suffix}_wheel_joint" type="continuous">
       <axis xyz="0 1 0"/>
-      <parent link="${prefix}_${suffix}_disk_wheel"/>
+      <parent link="${parent_link}"/>
       <child link="${prefix}_${suffix}_wheel"/>
       <origin xyz="${x} ${y} ${z}"/>
@@ -44,32 +56,32 @@
   </xacro:macro>
   <!-- Disk wheel -->
-<xacro:macro name="disk_wheel" params="prefix suffix roll pitch yaw with_gazebo:=false">
-  <link name="${prefix}_${suffix}_disk_wheel">
-    <visual>
-      <origin xyz="0 0 0" rpy="${roll} ${pitch} ${yaw}"/>
-      <geometry>
-        <mesh filename="$(arg pkg_share)//meshes/disk.dae" scale="1 1 1"/>
-      </geometry>
-    </visual>
-    <collision>
-      <geometry>
-        <cylinder radius="${disk_radius}" length="${disk_length}"/>
-      </geometry>
-      <origin xyz="0 0 0" rpy="1.5707 0 0"/>
-    </collision>
-    <inertial>
-      <mass value="${disk_mass}"/>
-      <origin xyz="0 0 0"/>
-      <inertia ixx="1.0" ixy="0" ixz="0" iyy="1.0" iyz="0" izz="1.0"/>
-    </inertial>
-  </link>
-  <xacro:if value="${with_gazebo}">
-    <gazebo reference="${prefix}_${suffix}_disk_wheel">
-      <material>Gazebo/Green</material>
-      <mu1>0.8</mu1>
-      <mu2>0.8</mu2>
-    </gazebo>
-  </xacro:if>
-</xacro:macro>
+  <xacro:macro name="disk_wheel" params="prefix suffix roll pitch yaw with_gazebo:=false">
+    <link name="${prefix}_${suffix}_disk_wheel">
+      <visual>
+        <origin xyz="0 0 0" rpy="${roll} ${pitch} ${yaw}"/>
+        <geometry>
+          <mesh filename="$(arg pkg_share)//meshes/disk.dae" scale="1 1 1"/>
+        </geometry>
+      </visual>
+      <collision>
+        <geometry>
+          <cylinder radius="${disk_radius}" length="${disk_length}"/>
+        </geometry>
+        <origin xyz="0 0 0" rpy="1.5707 0 0"/>
+      </collision>
+      <inertial>
+        <mass value="${disk_mass}"/>
+        <origin xyz="0 0 0"/>
+        <inertia ixx="1.0" ixy="0" ixz="0" iyy="1.0" iyz="0" izz="1.0"/>
+      </inertial>
+    </link>
+    <xacro:if value="${with_gazebo}">
+      <gazebo reference="${prefix}_${suffix}_disk_wheel">
+        <material>Gazebo/Green</material>
+        <mu1>0.8</mu1>
+        <mu2>0.8</mu2>
+      </gazebo>
+    </xacro:if>
+  </xacro:macro>
   <!-- Disk joint (front) -->
   <xacro:macro name="front_disk_wheel_joint" params="prefix suffix x y z">
@@ -79,6 +91,6 @@
       <origin xyz="${x} ${y} ${z}"/>
       <axis xyz="0 0 1"/>
-      <limit effort="1000.0" lower="-0.4" upper="0.4" velocity="0.5"/>
-      <dynamics damping="10.0" friction="1.0"/>
+      <limit effort="1000.0" lower="-0.523" upper="0.523" velocity="1.0"/>
+      <dynamics damping="0.1" friction="0.1"/>
       <initial_position>0.0</initial_position>
     </joint>

Commit message: Make local canonical: update bridge to km/h & deg, refine launch sequencing, add .gitignore

File: src/erp42_description/urdf/erp42.urdf.xacro (robot description, xacro)
@@ -5,4 +5,22 @@
   <xacro:include filename="$(arg pkg_share)/urdf/macros_erp42.xacro"/>
   <xacro:include filename="$(arg pkg_share)/urdf/erp42_control.gazebo" />
+  <link name="super_root"/>
+  <joint name="super_to_base_dummy" type="fixed">
+    <parent link="super_root"/>
+    <child link="base_dummy"/>
+    <origin xyz="0 0 0" rpy="0 0 0"/>
+  </joint>
+  <link name="base_dummy">
+    <inertial>
+      <mass value="160"/>
+      <origin xyz="0 0 0"/>
+      <inertia ixx="20.43" ixy="0.584" ixz="-0.191" iyy="54.197" iyz="-0.2449" izz="72.2588"/>
+    </inertial>
+  </link>
+  <joint name="base_dummy_to_structure" type="fixed">
+    <parent link="base_dummy"/>
+    <child link="structure"/>
+    <origin xyz="0 0 0" rpy="0 0 0"/>
+  </joint>
   <link name="structure">
     <visual name="visual">
@@ -18,9 +36,5 @@
       <origin xyz="0 0 -0.03" rpy="0 0 3.14" />
     </collision>
-    <inertial>
-      <mass value="160"/>
-      <origin xyz="0 0 0" />
-      <inertia ixx="20.43" ixy="0.584" ixz="-0.191" iyy="54.197" iyz="-0.2449" izz="72.2588"/>
-    </inertial>
+    <!-- removed inertia here; it's on base_dummy -->
   </link>
   <!-- steering links with visual for debug -->
@@ -118,7 +132,7 @@
         </clip>
       </camera>
-      <plugin name="camera_controller" filename="libgazebo_ros_camera.so">
-        <alwaysOn>true</alwaysOn>
-        <updateRate>0.0</updateRate>
+      <plugin name="left_camera_controller" filename="libgazebo_ros_camera.so">
+        <alwaysOn>true</alwaysOn>
+        <updateRate>30.0</updateRate>
         <cameraName>/erp42/left_camera</cameraName>
         <imageTopicName>image_raw</imageTopicName>
@@ -154,7 +168,7 @@
         </clip>
       </camera>
-      <plugin name="camera_controller" filename="libgazebo_ros_camera.so">
-        <alwaysOn>true</alwaysOn>
-        <updateRate>0.0</updateRate>
+      <plugin name="right_camera_controller" filename="libgazebo_ros_camera.so">
+        <alwaysOn>true</alwaysOn>
+        <updateRate>30.0</updateRate>
         <cameraName>/erp42/right_camera</cameraName>
         <imageTopicName>image_raw</imageTopicName>
@@ -190,7 +204,7 @@
         </clip>
       </camera>
-      <plugin name="camera_controller" filename="libgazebo_ros_camera.so">
-        <alwaysOn>true</alwaysOn>
-        <updateRate>0.0</updateRate>
+      <plugin name="middle_camera_controller" filename="libgazebo_ros_camera.so">
+        <alwaysOn>true</alwaysOn>
+        <updateRate>30.0</updateRate>
         <cameraName>/erp42/middle_camera</cameraName>
         <imageTopicName>image_raw</imageTopicName>
@@ -226,7 +240,7 @@
         </clip>
       </camera>
-      <plugin name="camera_controller" filename="libgazebo_ros_camera.so">
-        <alwaysOn>true</alwaysOn>
-        <updateRate>0.0</updateRate>
+      <plugin name="back_camera_controller" filename="libgazebo_ros_camera.so">
+        <alwaysOn>true</alwaysOn>
+        <updateRate>30.0</updateRate>
         <cameraName>/erp42/back_camera</cameraName>
         <imageTopicName>image_raw</imageTopicName>
